File: midi_glock_pcb/_restore_backup_2026-08-16T12-42-56-094/midi_glock_pcb.kicad_sch (KiCad schematic)
At the start: 52 parts, among them J1 Conn_01x12_Pin, J2 Conn_01x24_Pin, J3 Jack-DC, J4 Conn_01x06_Pin, J5 solenoid_return, J6 DM3D-SF, J7 Conn_01x04_Pin, U1 DRV8912QPWPRQ1, U2 DRV8912QPWPRQ1, U3 DRV8912QPWPRQ1, U4 LMR50410Y3FQDBVRQ1, U5 ESP32-WROVER-E-N4R8

Commit message: pcb almost complete
Parts:
- removed C20, C21, C22: 10uF, Capacitor_SMD:C_1206_3216Metric, symbol Device:C
- C1, C14, C15, C18, C2, C3, C4, C5, C6: footprint Capacitor_SMD:C_0603_1608Metric_Pad1.08x0.95mm_HandSolder -> Capacitor_SMD:C_0805_2012Metric_Pad1.18x1.45mm_HandSolder
- C10, C11, C12: footprint Capacitor_SMD:C_1206_3216Metric -> Capacitor_SMD:C_0805_2012Metric_Pad1.18x1.45mm_HandSolder
- C13, C17, C19: footprint Capacitor_SMD:C_1210_3225Metric -> Capacitor_SMD:C_0805_2012Metric_Pad1.18x1.45mm_HandSolder
- R1, R10, R11, R12, R2, R3, R4, R5, R6, R7, R8, R9: footprint Resistor_SMD:R_0603_1608Metric_Pad0.98x0.95mm_HandSolder -> Resistor_SMD:R_0805_2012Metric_Pad1.20x1.40mm_HandSolder
Connections:
- net DRV_nFAULT: now also U5.10 (IO25); no longer U5.33 (IO21)
- net DRV_nSLEEP: now also U5.11 (IO26); no longer U5.36 (IO22)
- net S1: now also J1.12 (Pin_12); no longer J1.4 (Pin_4)
- net S10: now also J1.3 (Pin_3); no longer J1.1 (Pin_1)
- net S11: now also J1.2 (Pin_2); no longer J1.6 (Pin_6)
- net S12: now also J1.1 (Pin_1); no longer J1.7 (Pin_7)
- net S13: now also J2.16 (Pin_16); no longer J2.15 (Pin_15)
- net S14: now also J2.15 (Pin_15); no longer J2.16 (Pin_16)
- net S15: now also J2.14 (Pin_14); no longer J2.17 (Pin_17)
- net S16: now also J2.21 (Pin_21); no longer J2.22 (Pin_22)
- net S17: now also J2.17 (Pin_17); no longer J2.14 (Pin_14)
- net S18: now also J2.22 (Pin_22); no longer J2.21 (Pin_21)
- net S19: now also J2.20 (Pin_20); no longer J2.19 (Pin_19)
- net S2: now also J1.11 (Pin_11); no longer J1.3 (Pin_3)
- net S21: now also J2.19 (Pin_19); no longer J2.20 (Pin_20)
- net S22: now also J2.13 (Pin_13); no longer J2.18 (Pin_18)
- net S23: now also J2.18 (Pin_18); no longer J2.13 (Pin_13)
- net S25: now also J2.12 (Pin_12); no longer J2.10 (Pin_10)
- net S26: now also J2.11 (Pin_11); no longer J2.9 (Pin_9)
- net S27: now also J2.10 (Pin_10); no longer J2.12 (Pin_12)
- net S28: now also J2.9 (Pin_9); no longer J2.3 (Pin_3)
- net S29: now also J2.8 (Pin_8); no longer J2.7 (Pin_7)
- net S3: now also J1.10 (Pin_10); no longer J1.2 (Pin_2)
- net S30: now also J2.7 (Pin_7); no longer J2.4 (Pin_4)
- net S31: now also J2.6 (Pin_6); no longer J2.2 (Pin_2)
- net S33: now also J2.4 (Pin_4); no longer J2.1 (Pin_1)
- net S34: now also J2.3 (Pin_3); no longer J2.11 (Pin_11)
- net S35: now also J2.2 (Pin_2); no longer J2.8 (Pin_8)
- net S36: now also J2.1 (Pin_1); no longer J2.6 (Pin_6)
- net S4: now also J1.9 (Pin_9); no longer J1.10 (Pin_10)
- net S5: now also J1.8 (Pin_8); no longer J1.5 (Pin_5)
- net S6: now also J1.7 (Pin_7); no longer J1.9 (Pin_9)
- net S7: now also J1.6 (Pin_6); no longer J1.11 (Pin_11)
- net S8: now also J1.5 (Pin_5); no longer J1.8 (Pin_8)
- net S9: now also J1.4 (Pin_4); no longer J1.12 (Pin_12)
Other:
- moved on the sheet: C17, C18, L1, U4
