File: midi_glock_pcb/midi_glock_pcb.kicad_sch (KiCad schematic)
At the start: 52 parts, among them J1 Conn_01x12_Pin, J2 Conn_01x24_Pin, J3 Jack-DC, J4 Conn_01x06_Pin, J5 solenoid_return, J6 DM3D-SF, J7 Conn_01x04_Pin, U1 DRV8912QPWPRQ1, U2 DRV8912QPWPRQ1, U3 DRV8912QPWPRQ1, U4 LMR50410Y3FQDBVRQ1, U5 ESP32-WROVER-E-N4R8

Commit message: added test points
Parts:
- added TP1: MOSI, TestPoint:TestPoint_Pad_D1.0mm, symbol Connector:TestPoint
- added TP2: MISO, TestPoint:TestPoint_Pad_D1.0mm, symbol Connector:TestPoint
- added TP3: CS, TestPoint:TestPoint_Pad_D1.0mm, symbol Connector:TestPoint
- added TP4: CLK, TestPoint:TestPoint_Pad_D1.0mm, symbol Connector:TestPoint
Connections:
- net SPI_CS: now also TP3.1
- net SPI_MISO: now also TP2.1
- net SPI_MOSI: now also TP1.1
- net SPI_SCLK: now also TP4.1
Other:
- note removed: "Todo: - Derate caps"
