File: midi_glock_pcb/midi_glock_pcb.kicad_pcb (KiCad board)
At the start: 4 copper layers, 52 x 90.3 mm, 59 parts, among them J1 Conn_01x12_Pin, J2 Conn_01x24_Pin, J3 Jack-DC, J4 Conn_01x06_Pin, J5 solenoid_return, J6 DM3D-SF, J7 Conn_01x04_Pin, U1 DRV8912QPWPRQ1, U2 DRV8912QPWPRQ1, U3 DRV8912QPWPRQ1, U4 LMR50410Y3FQDBVRQ1, U5 ESP32-WROVER-E-N4R8

Commit message: fixed misc grounds on layout
Parts:
- REF** (x3): value MountingHole_3.2mm_M3_DIN965_Pad_TopBottom -> MountingHole_3.2mm_M3_DIN965_Pad; footprint MountingHole:MountingHole_3.2mm_M3_DIN965_Pad_TopBottom -> MountingHole:MountingHole_3.2mm_M3_DIN965_Pad
- moved REF** 0.78 mm to (94.9, 88.5)
Routing:
- net GND: track 128.6 -> 132.1 mm, vias 81 -> 106
